Commit message: urdf comp.

File: robocup_ws/src/robot_description/description/robot_description_test.urdf (robot description, URDF)
Before this commit: robot amr, 7 links, 6 joints
Links:
- link chassis: geometry collision box size=0.225 0.36 0.61; visual box size=0.225 0.36 0.61
- link wheel_left_link: geometry collision cylinder length=0.046 radius=0.085; visual cylinder length=0.046 radius=0.085
- link wheel_right_link: geometry collision cylinder length=0.046 radius=0.085; visual cylinder length=0.046 radius=0.085
