Commit message: urdf comp.

File: robocup_ws/src/robot_description/description/robot_description.urdf (robot description, URDF)
Before this commit: robot amr, 8 links, 7 joints
Links:
- removed link imu_link
- link chassis: geometry visual box size=0.72 0.45 0.61
- link wheel_left_link: geometry collision cylinder length=0.046 radius=0.085; visual cylinder length=0.046 radius=0.085
- link wheel_right_link: geometry collision cylinder length=0.046 radius=0.085; visual cylinder length=0.046 radius=0.085
Joints:
- removed joint imu_joint
- joint base_joint: origin xyz=0 0 0.2175 rpy=0 0 0 -> xyz=0 0 0.001 rpy=0 0 0
- joint lidar1_joint: origin xyz=0.105 -0.075 0.13 rpy=0 0 0 -> xyz=0.345 0.0 0.04 rpy=0. 0 -1.57
- joint lidar2_joint: origin xyz=-0.105 0.075 0.13 rpy=0 0 3.14159 -> xyz=-0.345 -0.0 0.04 rpy=0. 0 1.57
- joint lidar_joint: origin xyz=0.0 0.0 0.13 rpy=0 0 3.14 -> xyz=0.0 0.0 0.04 rpy=0 0 -1.57
- joint wheel_left_joint: axis 0 -1 0 -> (none); origin xyz=0.14 0.16 -0.1425 rpy=0 0 0 -> xyz=0 0.145 0.085 rpy=-1.57 0 0; type continuous -> fixed
- joint wheel_right_joint: axis 0 -1 0 -> (none); origin xyz=0.14 -0.16 -0.1425 rpy=0 0 0 -> xyz=0 -0.145 0.085 rpy=1.57 0 0; type continuous -> fixed

File: robocup_ws/src/robot_description/description/robot_description_test.urdf (robot description, URDF)
Before this commit: robot amr, 7 links, 6 joints
Links:
- link chassis: geometry visual box size=0.72 0.45 0.61
Joints:
- joint lidar1_joint: origin xyz=0.24698 0.143555 0.2 rpy=0. 0 -1.57 -> xyz=0.345 0.0 0.04 rpy=0. 0 -1.57
- joint lidar2_joint: origin xyz=-0.24698 -0.143555 0.2 rpy=0. 0 1.57 -> xyz=-0.345 -0.0 0.04 rpy=0. 0 1.57
- joint lidar_joint: origin xyz=0.0 0.0 0.2 rpy=0 0 -1.57 -> xyz=0.0 0.0 0.04 rpy=0 0 -1.57

Commit message: lidar urdf update (test)

File: robocup_ws/src/robot_description/description/robot_description.urdf (robot description, URDF)
Before this commit: robot amr, 7 links, 6 joints
Joints:
- joint lidar1_joint: origin xyz=0.345 0.0 0.04 rpy=0. 0 -1.57 -> xyz=0.345 0.0 0.04 rpy=3.14. 0 -3.14
- joint lidar2_joint: origin xyz=-0.345 -0.0 0.04 rpy=0. 0 1.57 -> xyz=-0.345 -0.0 0.04 rpy=3.14. 0 0
- joint lidar_joint: origin xyz=0.0 0.0 0.04 rpy=0 0 -1.57 -> xyz=0.0 0.0 0.04 rpy=3.14 0 -3.14

Commit message: lidar urdf update (test)

File: robocup_ws/src/robot_description/description/robot_description.urdf (robot description, URDF)
Before this commit: robot amr, 7 links, 6 joints
Joints:
- joint lidar1_joint: origin xyz=0.345 0.0 0.04 rpy=3.14. 0 -3.14 -> xyz=0.345 0.0 0.04 rpy=3.14 0 -3.14
- joint lidar2_joint: origin xyz=-0.345 -0.0 0.04 rpy=3.14. 0 0 -> xyz=-0.345 -0.0 0.04 rpy=3.14 0 0

Commit message: lidar urdf update (test)

File: robocup_ws/src/robot_description/description/robot_description.urdf (robot description, URDF)
Before this commit: robot amr, 7 links, 6 joints
Joints:
- joint lidar1_joint: origin xyz=0.345 0.0 0.04 rpy=3.14 0 -3.14 -> xyz=-0.345 -0.0 0.04 rpy=3.14 0 0
- joint lidar2_joint: origin xyz=-0.345 -0.0 0.04 rpy=3.14 0 0 -> xyz=0.345 0.0 0.04 rpy=3.14 0 -3.14

Commit message: lidar urdf update (test)

File: robocup_ws/src/robot_description/description/robot_description.urdf (robot description, URDF)
Before this commit: robot amr, 7 links, 6 joints
Joints:
- joint lidar1_joint: origin xyz=-0.345 -0.0 0.04 rpy=3.14 0 0 -> xyz=0.345 0.0 0.04 rpy=3.14 0 -3.14
- joint lidar2_joint: origin xyz=0.345 0.0 0.04 rpy=3.14 0 -3.14 -> xyz=-0.345 -0.0 0.04 rpy=3.14 0 0

Commit message: wheel dyn urdf update (test)

File: robocup_ws/src/robot_description/description/robot_description.urdf (robot description, URDF)
Before this commit: robot amr, 7 links, 6 joints
Joints:
- joint wheel_left_joint: axis (none) -> 0 0 1; type fixed -> continuous
- joint wheel_right_joint: axis (none) -> 0 0 1; type fixed -> continuous
